Commit message: Linkus: sensors, msgs, nav params

File: rover_description/robots/rover.urdf.xacro (robot description, xacro)
@@ -177,15 +177,29 @@
     <xacro:bogie lat_label="right" reflect="-1"/>
     <!-- sensors -->
-    <xacro:sensor_hokuyo prefix="laser" parent="base_link" min_angle="-1.0" max_angle="1.0">
-        <origin xyz="0.17 0 0.005" rpy="0 0 0"/>
-    </xacro:sensor_hokuyo>
-    <xacro:sensor_imu prefix="imu" parent="base_link">
-        <!-- <origin xyz="-0.32 0 0.05" rpy="0 0.5 0"/> -->
-        <origin xyz="0 0 -0.04" rpy="0 0 0"/>
-    </xacro:sensor_imu>
-    <xacro:sensor_asus_xtion prefix="camera" parent="base_link">
-        <origin xyz="0.215 0 0.065" rpy="0 0.4 0"/>
-        <!-- <origin xyz="0.212 0 0.065" rpy="0 0 0"/> -->
-    </xacro:sensor_asus_xtion>
+    <!--
+      MOUNTING POSES LIVE HERE AND ONLY HERE.
+      The <origin> of each sensor below is the single source of truth for
+      where that sensor sits on the rover. Everything downstream (rtabmap,
+      robot_localization, nav2, RViz) works off TF, so changing a pose needs
+      no edit anywhere else.
+      Two things that are NOT poses and do live elsewhere:
+        * Link names (laser_link, imu_link, camera_*) are referenced by
+          frame_id in rover_bringup/config/*.yaml - keep them as they are.
+        * If the RPLIDAR C1 ends up mounted upside down, set inverted: true
+          in rover_bringup/config/rplidar_c1.yaml as well; the driver, not
+          the URDF, is what reverses the scan direction on real hardware.
+    -->
+    <!-- Slamtec RPLIDAR C1: full 360 deg scan, 0.05-12 m -->
+    <xacro:sensor_rplidar_c1 prefix="laser" parent="base_link">
+        <origin xyz="0.17 -0.047 0.033" rpy="0 0 3.14159265"/>
+    </xacro:sensor_rplidar_c1>
+    <!-- Adafruit BNO085 9-DOF IMU -->
+    <xacro:sensor_bno085 prefix="imu" parent="base_link">
+        <origin xyz="-0.17 0 0" rpy="0 0 -1.5708"/>
+    </xacro:sensor_bno085>
+    <!-- Orbbec Gemini 335 RGB-D camera -->
+    <xacro:sensor_gemini_335 prefix="camera" parent="base_link">
+        <origin xyz="0.17 0.047 0.205" rpy="0 0 0"/>
+    </xacro:sensor_gemini_335>
     <!-- wheels -->
     <xacro:corner_link lon_label="front" lat_label="left" reflect="1"/>

File: rover_description/urdf/sensors/all_sensors.urdf.xacro (robot description, xacro)
@@ -18,9 +18,9 @@
 # SOFTWARE. -->
 <robot name="all_sensors" xmlns:xacro="http://www.ros.org/wiki/xacro">
-  <!-- Imu -->
-  <xacro:include filename="$(find rover_description)/urdf/sensors/imu.urdf.xacro" />
-  <!-- Hokuyo -->
-  <xacro:include filename="$(find rover_description)/urdf/sensors/hokuyo.urdf.xacro" />
-  <!-- Hokuyo -->
-  <xacro:include filename="$(find rover_description)/urdf/sensors/asus_xtion.urdf.xacro" />
+  <!-- IMU: Adafruit BNO085 9-DOF -->
+  <xacro:include filename="$(find rover_description)/urdf/sensors/bno085.urdf.xacro" />
+  <!-- 2D lidar: Slamtec RPLIDAR C1 -->
+  <xacro:include filename="$(find rover_description)/urdf/sensors/rplidar_c1.urdf.xacro" />
+  <!-- RGB-D camera: Orbbec Gemini 335 -->
+  <xacro:include filename="$(find rover_description)/urdf/sensors/gemini_335.urdf.xacro" />
 </robot>

File: rover_description/urdf/sensors/bno085.urdf.xacro (robot description, xacro)
@@ -1,5 +1,5 @@
 <?xml version="1.0" ?>
 <!-- # MIT License
-# Copyright (c) 2023 Miguel Ángel González Santamarta
+# Copyright (c) 2023  Miguel Ángel González Santamarta
 # Permission is hereby granted, free of charge, to any person obtaining a copy
 # of this software and associated documentation files (the "Software"), to deal
@@ -17,29 +17,37 @@
 # OUT OF OR IN CONNECTION WITH THE SOFTWARE OR THE USE OR OTHER DEALINGS IN THE
 # SOFTWARE. -->
-<robot name="sensor_imu" xmlns:xacro="http://www.ros.org/wiki/xacro">
-  <xacro:macro name="sensor_imu" params="prefix parent *origin">
+<!-- Adafruit BNO085 9-DOF Orientation IMU breakout (CEVA/Hillcrest BNO08x).
+     Breakout board 25.4 x 17.8 x 3 mm, driven over I2C by bno08x_driver.
+     Noise figures below come from the BNO080/BNO085 datasheet:
+       gyro  0.014 deg/s/sqrt(Hz) -> 2.4e-4 rad/s/sqrt(Hz)
+       accel 190 ug/sqrt(Hz)      -> 1.9e-3 m/s^2/sqrt(Hz)
+     scaled to the 100 Hz report rate configured in
+     rover_bringup/config/bno085.yaml.
+     Gazebo Classic version: published by libgazebo_ros_imu_sensor. -->
+<robot name="sensor_bno085" xmlns:xacro="http://www.ros.org/wiki/xacro">
+  <xacro:macro name="sensor_bno085" params="prefix parent *origin update_rate:=100">
     <joint name="${prefix}_joint" type="fixed">
-      <axis xyz="1 0 0"/>
-      <xacro:insert_block name="origin"/>
-      <parent link="${parent}"/>
-      <child link="${prefix}_link"/>
+      <axis xyz="1 0 0" />
+      <xacro:insert_block name="origin" />
+      <parent link="${parent}" />
+      <child link="${prefix}_link" />
     </joint>
     <link name="${prefix}_link">
       <inertial>
-        <mass value="0.001"/>
-        <origin rpy="0 0 0" xyz="0 0 0"/>
-        <inertia ixx="0.0001" ixy="0" ixz="0" iyy="0.000001" iyz="0" izz="0.0001"/>
+        <mass value="0.003" />
+        <origin rpy="0 0 0" xyz="0 0 0" />
+        <inertia ixx="8e-8" ixy="0" ixz="0" iyy="1.6e-7" iyz="0" izz="2.4e-7" />
       </inertial>
       <visual>
-        <origin rpy="0 0 0" xyz="0 0 0"/>
+        <origin rpy="0 0 0" xyz="0 0 0" />
         <geometry>
-          <box size="0.03 0.02 0.01"/>
+          <box size="0.0254 0.0178 0.003" />
         </geometry>
         <material name="blue" />
       </visual>
       <collision>
-        <origin rpy="0 0 0" xyz="0 0 0"/>
+        <origin rpy="0 0 0" xyz="0 0 0" />
         <geometry>
-          <box size=".001 .001 .001"/>
+          <box size="0.0254 0.0178 0.003" />
         </geometry>
       </collision>
@@ -49,6 +57,6 @@
     </gazebo>
     <gazebo reference="${prefix}_link">
-      <sensor name="imu_sensor" type="imu">
-        <plugin filename="libgazebo_ros_imu_sensor.so" name="imu_controller">
+      <sensor name="bno085" type="imu">
+        <plugin filename="libgazebo_ros_imu_sensor.so" name="${prefix}_controller">
           <ros>
             <remapping>~/out:=imu</remapping>
@@ -65,5 +73,5 @@
         </plugin>
         <always_on>true</always_on>
-        <update_rate>200</update_rate>
+        <update_rate>${update_rate}</update_rate>
         <visualize>true</visualize>
         <imu>
@@ -72,5 +80,5 @@
               <noise type="gaussian">
                 <mean>0.0</mean>
-                <stddev>2e-4</stddev>
+                <stddev>2.4e-3</stddev>
                 <bias_mean>0.0000075</bias_mean>
                 <bias_stddev>0.0000008</bias_stddev>
@@ -80,5 +88,5 @@
               <noise type="gaussian">
                 <mean>0.0</mean>
-                <stddev>2e-4</stddev>
+                <stddev>2.4e-3</stddev>
                 <bias_mean>0.0000075</bias_mean>
                 <bias_stddev>0.0000008</bias_stddev>
@@ -88,5 +96,5 @@
               <noise type="gaussian">
                 <mean>0.0</mean>
-                <stddev>2e-4</stddev>
+                <stddev>2.4e-3</stddev>
                 <bias_mean>0.0000075</bias_mean>
                 <bias_stddev>0.0000008</bias_stddev>
@@ -98,5 +106,5 @@
               <noise type="gaussian">
                 <mean>0.0</mean>
-                <stddev>1.7e-2</stddev>
+                <stddev>1.9e-2</stddev>
                 <bias_mean>0.1</bias_mean>
                 <bias_stddev>0.001</bias_stddev>
@@ -106,5 +114,5 @@
               <noise type="gaussian">
                 <mean>0.0</mean>
-                <stddev>1.7e-2</stddev>
+                <stddev>1.9e-2</stddev>
                 <bias_mean>0.1</bias_mean>
                 <bias_stddev>0.001</bias_stddev>
@@ -114,5 +122,5 @@
               <noise type="gaussian">
                 <mean>0.0</mean>
-                <stddev>1.7e-2</stddev>
+                <stddev>1.9e-2</stddev>
                 <bias_mean>0.1</bias_mean>
                 <bias_stddev>0.001</bias_stddev>

File: rover_description/urdf/sensors/rplidar_c1.urdf.xacro (robot description, xacro)
@@ -1,5 +1,5 @@
 <?xml version="1.0" ?>
 <!-- # MIT License
-# Copyright (c) 2023 Miguel Ángel González Santamarta
+# Copyright (c) 2023  Miguel Ángel González Santamarta
 # Permission is hereby granted, free of charge, to any person obtaining a copy
 # of this software and associated documentation files (the "Software"), to deal
@@ -17,49 +17,56 @@
 # OUT OF OR IN CONNECTION WITH THE SOFTWARE OR THE USE OR OTHER DEALINGS IN THE
 # SOFTWARE. -->
-<robot name="sensor_hokuyo" xmlns:xacro="http://www.ros.org/wiki/xacro">
-  <xacro:macro name="sensor_hokuyo" params="prefix parent *origin min_angle:=-1.57079637051 max_angle:=1.57079637051">
-    <joint name="${prefix}_base_joint" type="fixed">
+<!-- Slamtec RPLIDAR C1 (360 deg DTOF, 0.05-12 m, 10 Hz, 5000 samples/s)
+     Gazebo Classic version: the scan is published by libgazebo_ros_ray_sensor. -->
+<robot name="sensor_rplidar_c1" xmlns:xacro="http://www.ros.org/wiki/xacro">
+  <xacro:macro name="sensor_rplidar_c1" params="prefix parent *origin
+                                                min_angle:=${-pi} max_angle:=${pi}
+                                                samples:=500 update_rate:=10
+                                                min_range:=0.05 max_range:=12.0">
+    <!-- Housing: 55.6 x 55.6 x 41.3 mm. The scan plane sits ~28 mm above the
+         base, so the body is drawn slightly below ${prefix}_link, which IS the
+         scan frame (matches the driver's frame_id). -->
+    <xacro:property name="rplidar_radius" value="0.0278" />
+    <xacro:property name="rplidar_height" value="0.0413" />
+    <xacro:property name="rplidar_visual_z" value="-0.0074" />
+    <joint name="${prefix}_joint" type="fixed">
       <xacro:insert_block name="origin" />
-      <parent link="${parent}"/>
-      <child link="${prefix}_base_link"/>
+      <parent link="${parent}" />
+      <child link="${prefix}_link" />
     </joint>
-    <link name="${prefix}_base_link">
+    <link name="${prefix}_link">
+      <visual>
+        <origin xyz="0 0 ${rplidar_visual_z}" rpy="0 0 0" />
+        <geometry>
+          <cylinder radius="${rplidar_radius}" length="${rplidar_height}" />
+        </geometry>
+        <material name="dark_gray" />
+      </visual>
       <collision>
-        <origin xyz="0 0 -0.05" rpy="0 0 0"/>
+        <origin xyz="0 0 ${rplidar_visual_z}" rpy="0 0 0" />
         <geometry>
-          <box size="0.010 0.010 0.010"/>
+          <cylinder radius="${rplidar_radius}" length="${rplidar_height}" />
         </geometry>
       </collision>
-      <visual>
-        <origin xyz="0 0 -0.05" rpy="0 0 0"/>
-        <geometry>
-          <mesh filename="package://rover_description/meshes/sensors/hokuyo/hokuyo_ust_20lx.dae"/>
-        </geometry>
-      </visual>
       <inertial>
-        <mass value="1e-5" />
-        <origin xyz="0 0 0" rpy="0 0 0"/>
-        <inertia ixx="1e-6" ixy="0" ixz="0" iyy="1e-6" iyz="0" izz="1e-6" />
+        <mass value="0.11" />
+        <origin xyz="0 0 ${rplidar_visual_z}" rpy="0 0 0" />
+        <inertia ixx="2.1e-5" ixy="0" ixz="0" iyy="2.1e-5" iyz="0" izz="4.2e-5" />
       </inertial>
     </link>
-    <gazebo reference="${prefix}_base_link">
+    <gazebo reference="${prefix}_link">
       <material>Gazebo/DarkGrey</material>
     </gazebo>
-    <link name="${prefix}_link">
-    </link>
-    <joint name="${prefix}_joint" type="fixed">
-      <parent link="${prefix}_base_link"/>
-      <child link="${prefix}_link"/>
-      <origin xyz="0.00 0 0.0" rpy="0 0 0"/>
-    </joint>
     <gazebo reference="${prefix}_link">
-      <sensor type="gpu_ray" name="hokuyo_sensor">
+      <sensor name="rplidar_c1" type="gpu_ray">
         <pose>0 0 0 0 0 0</pose>
+        <always_on>true</always_on>
         <visualize>true</visualize>
-        <update_rate>50</update_rate>
+        <update_rate>${update_rate}</update_rate>
         <ray>
           <scan>
             <horizontal>
-              <samples>30</samples>
+              <!-- 5000 samples/s at 10 Hz => 500 samples/turn (0.72 deg) -->
+              <samples>${samples}</samples>
               <resolution>1</resolution>
               <min_angle>${min_angle}</min_angle>
@@ -68,7 +75,8 @@
           </scan>
           <range>
-            <min>0.06</min>
-            <max>5.0</max>
-            <resolution>0.004359297</resolution>
+            <min>${min_range}</min>
+            <max>${max_range}</max>
+            <!-- Datasheet accuracy: +-30 mm -->
+            <resolution>0.03</resolution>
           </range>
           <noise>
